File: PCB/MainBoard/MainBoard.kicad_sch (KiCad schematic)
At the start: 18 parts, among them J10 Conn_01x06_Socket, J11 Conn_01x06_Socket, J12 Conn_01x04_Socket, J18 Conn_01x04_Socket, J19 Conn_01x04_Socket, J20 Conn_01x04_Socket, J5 Conn_01x03_Socket, J6 Conn_01x03_Socket, J7 Conn_01x03_Socket, SW1 SW_Push, U3 STM32F103C8Tx

Commit message: adding board v2 progress
Parts:
- added C22, C24, C26, C27, C28: 100n, Capacitor_SMD:C_0603_1608Metric, symbol basic:C
- added C23: 10n, Capacitor_SMD:C_0603_1608Metric, symbol basic:C
- added C25, C30: 1u, Capacitor_SMD:C_0603_1608Metric, symbol basic:C
- added C29: 4.7u, Capacitor_SMD:C_0603_1608Metric, symbol basic:C
- added R11: 10k, Resistor_SMD:R_0603_1608Metric, symbol basic:R
- added SW2: SW_Push, Button_Switch_SMD:SW_SPST_B3S-1000, symbol Switch:SW_Push
- added TP7: 3V3, TestPoint:TestPoint_Keystone_5000-5004_Miniature, symbol Connector:TestPoint
- U3: value STM32F103C8Tx -> STM32F103C8T6TR
Connections:
- net +3.3V_1.2A is gone; now on net +3V3: J18.1 (Pin_1), J19.1 (Pin_1), J20.1 (Pin_1), U3.24 (VDD), U3.36 (VDD), U3.48 (VDD), U3.9 (VDDA)
- net GND: now also C22.2, C23.2, C24.2, C25.2, C26.2, C27.2, C28.2, C29.2, C30.2, SW2.1
- net LimitSwitchORGates/OR3 Output: no longer U3.22 (PB11)
- net ME1_ChA: no longer U3.12 (PA2)
- net ME1_ChB: no longer U3.13 (PA3)
- net ME2_ChA: no longer U3.18 (PB0)
- net ME2_ChB: no longer U3.19 (PB1)
- net ME3_ChA: no longer U3.16 (PA6)
- net ME3_ChB: no longer U3.17 (PA7)
- net SPI2_MISO: no longer U3.27 (PB14)
- net SPI2_MOSI: no longer U3.28 (PB15)
- net SPI2_NSS: no longer U3.25 (PB12)
- net SPI2_SCK: no longer U3.26 (PB13)
- net at C5.1, SW1.2: no longer U3.7 (NRST)
- net +3V3: now reaches U3.1 (VBAT)
- net +3V3: now also C22.1, C23.1, C24.1, C25.1, C26.1, C27.1, C28.1, C29.1, R11.1, TP7.1
- net at U3.21 (PB10): no longer J7.3 (Pin_3)
- net at U3.39 (PB3): no longer J5.3 (Pin_3)
- net at U3.40 (PB4): no longer J6.3 (Pin_3)
- new net NRST: C30.1, R11.2, SW2.2, U3.7 (NRST)
- no-connect marks 25 -> 24
Other:
- note added: "Connect 4.7u cap to V_dd3 (pin 48)"
- moved on the sheet: C3, C4, C5, H1, H2, H3, H4, J10, J11, J12, J18, J19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

Commit message: updating main board v2 with motor power conns
Other:
- moved on the sheet: C3, C4, H1, H2, H3, H4, J10, J11, J12, J18, J19, J20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
