File: PCB/MainBoardv2.1/MainBoardv2_1/MainBoardv2_1.kicad_pcb (KiCad board)
At the start: 2 copper layers, 100 x 100 mm, 103 parts, among them J1 Conn_02x03_Odd_Even, J10 Conn_01x03_Socket, J11 Conn_01x03_Socket, J12 Conn_01x04_Socket, J13 Conn_01x03_Socket, J14 Conn_01x03_Socket, J15 Conn_01x04_Socket, J16 Conn_01x03_Socket, J17 Conn_01x03_Socket, J18 Conn_01x04_Socket, J19 Conn_01x03_Socket, J2 USB_B_Micro, J20 Screw_Terminal_01x02, J21 Screw_Terminal_01x02, J22 Screw_Terminal_01x02, J23 Conn_01x03_Socket, J24 Conn_01x03_Socket, J25 Conn_01x03_Socket, J3 Conn_02x03_Odd_Even, J4 Conn_01x05_Pin, J5 Screw_Terminal_01x02, J6 Conn_01x04_Socket, J7 Screw_Terminal_01x02, J8 Conn_01x04_Socket, J9 Conn_01x04_Socket, SW1 SW_Push, SW2 Toggle, SW3 Slide, U1 AZ1117-3.3, U2 STM32F103C8T6TR, U3 TPS56637RPA, U4 CD74HC00_N_14, U5 SN74HCS4075PWR, Y1 8MHz Crystal

Commit message: main board v2 sent to fab
Routing:
- net +3.3V: track 224.9 -> 117.7 mm, vias 18 -> 10
- net /TIM4_CH1: track 90.7 -> 1.99 mm, vias 9 -> 1
- net /TIM4_CH2: track 99.5 -> 16.6 mm, vias 12 -> 2
- net /TIM3_CH1: track 82.7 -> 0.00 mm, vias 3 -> 0
- net /TIM3_CH2: track 78.5 -> 0.00 mm, vias 2 -> 0
- net /TIM2_CH1: track 65.3 -> 0.00 mm, vias 1 -> 0
- net /TIM2_CH2: track 58.1 -> 1.25 mm
- net /TIM1_CH3: track 50.0 -> 0.00 mm, vias 1 -> 0
- net /TIM1_CH1: track 49.4 -> 0.00 mm, vias 2 -> 0
- net /TIM1_CH2: track 48.4 -> 0.00 mm, vias 4 -> 0
- net /PWM & Encoders & Limit Switches/M1_PWM: track 58.7 -> 11.1 mm, vias 2 -> 0
- net +12V: track 83.0 -> 40.1 mm
- net /OR3: track 45.4 -> 7.95 mm, vias 7 -> 0
- net /PWM & Encoders & Limit Switches/M2_PWM: track 48.1 -> 11.1 mm, vias 2 -> 0
- net /PWM & Encoders & Limit Switches/M3_PWM: track 45.4 -> 11.8 mm
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Other:
- board text removed: "3PDT"
